Commit message: 載入rs_m90e7_description 可使用 ros2 launch cool_robot_description view_cool_robot.launch.py 觀看機器人 在ros2_control架構加入rs_m90e7的ethercat master

File: cool_robot_description/urdf/cool_robot.urdf.xacro (robot description, xacro)
@@ -1,27 +1,20 @@
 <?xml version="1.0" encoding="UTF-8"?>
 <robot xmlns:xacro="http://wiki.ros.org/xacro" name="cool_robot">
-  <!-- Use this if parameters are set from the launch file, otherwise delete -->
-  <xacro:arg name="prefix" default="" />
-  <xacro:arg name="use_mock_hardware" default="false" />
-  <xacro:arg name="mock_sensor_commands" default="false" />
-  <xacro:arg name="sim_gazebo_classic" default="false" />
-  <xacro:arg name="sim_gazebo" default="false" />
-  <xacro:arg name="simulation_controllers" default="" />
-  <xacro:include filename="$(find cool_robot_description)/urdf/cool_robot/cool_robot_macro.xacro"/>
+  <!-- ========================================= -->
+  <!-- include macro from xacro files -->
+  <!-- ========================================= -->
+  <xacro:include filename="$(find rs_m90e7_description)/urdf/rs_m90e7/rs_m90e7_macro.xacro"/>
   <xacro:include filename="$(find cool_robot_description)/urdf/cool_robot/cool_robot_macro.ros2_control.xacro"/>
+  <!-- ========================================= -->
+  <!-- define robot-->
+  <!-- ========================================= -->
   <!-- create link fixed to the "world" -->
   <link name="world" />
-  <!-- Load robot's macro with parameters -->
-  <!-- set prefix if multiple robots are used -->
-  <xacro:cool_robot prefix="$(arg prefix)" parent="world" >
-    <origin xyz="0 0 0" rpy="0 0 0" />          <!-- position robot in the world -->
-  </xacro:cool_robot>
-  <xacro:cool_robot_ros2_control
-    name="cool_robot"
-    prefix="$(arg prefix)"
-    use_mock_hardware="$(arg use_mock_hardware)"
-    mock_sensor_commands="$(arg mock_sensor_commands)"
-    sim_gazebo_classic="$(arg sim_gazebo_classic)"
-    sim_gazebo="$(arg sim_gazebo)"
-    simulation_controllers="$(arg simulation_controllers)" />
+  <xacro:rs_m90e7 prefix="" parent="world">
+    <origin xyz="0.5 0 0" rpy="0 0 0" />
+  </xacro:rs_m90e7>
+  <!-- ========================================= -->
+  <!-- define ros2 control-->
+  <!-- ========================================= -->
+  <xacro:cool_robot_ros2_control name="cool_robot" prefix=""/>
 </robot>

File: cool_robot_description/urdf/cool_robot/cool_robot_macro.ros2_control.xacro (robot description, xacro)
@@ -3,29 +3,10 @@
   <xacro:macro name="cool_robot_ros2_control" params="
                name
-               prefix
-               use_mock_hardware:=^|false
-               mock_sensor_commands:=^|false
-               sim_gazebo_classic:=^|false
-               sim_gazebo:=^|false
-               simulation_controllers"
-               >
+               prefix">
     <ros2_control name="${name}" type="system">
       <hardware>
-        <xacro:if value="${use_mock_hardware}">
-          <plugin>mock_components/GenericSystem</plugin>
-          <param name="mock_sensor_commands">${mock_sensor_commands}</param>
-        </xacro:if>
-        <xacro:if value="${sim_gazebo_classic}">
-          <plugin>gazebo_ros2_control/GazeboSystem</plugin>
-        </xacro:if>
-        <xacro:if value="${sim_gazebo}">
-          <plugin>ign_ros2_control/IgnitionSystem</plugin>
-        </xacro:if>
-        <xacro:unless value="${use_mock_hardware or sim_gazebo_classic or sim_gazebo}">
-          <plugin>robot_hardware_inteface/RobotHardwareInteface</plugin>
-        </xacro:unless>
       </hardware>
       <joint name="${prefix}joint1">
-        <command_interface name="position">     <!-- Add/Remove interfaces as needed -->
+        <command_interface name="position">          <!-- Add/Remove interfaces as needed -->
           <param name="min">-1</param>
           <param name="max">1</param>
@@ -38,5 +19,5 @@
       </joint>
       <joint name="${prefix}joint2">
-        <command_interface name="position">     <!-- Add/Remove interfaces as needed -->
+        <command_interface name="position">          <!-- Add/Remove interfaces as needed -->
           <param name="min">-1</param>
           <param name="max">1</param>
@@ -49,5 +30,5 @@
       </joint>
       <joint name="${prefix}joint3">
-        <command_interface name="position">     <!-- Add/Remove interfaces as needed -->
+        <command_interface name="position">          <!-- Add/Remove interfaces as needed -->
           <param name="min">-1</param>
           <param name="max">1</param>
@@ -60,5 +41,5 @@
       </joint>
       <joint name="${prefix}joint4">
-        <command_interface name="position">     <!-- Add/Remove interfaces as needed -->
+        <command_interface name="position">          <!-- Add/Remove interfaces as needed -->
           <param name="min">-1</param>
           <param name="max">1</param>
@@ -71,5 +52,5 @@
       </joint>
       <joint name="${prefix}joint5">
-        <command_interface name="position">     <!-- Add/Remove interfaces as needed -->
+        <command_interface name="position">          <!-- Add/Remove interfaces as needed -->
           <param name="min">-1</param>
           <param name="max">1</param>
@@ -82,5 +63,5 @@
       </joint>
       <joint name="${prefix}joint6">
-        <command_interface name="position">     <!-- Add/Remove interfaces as needed -->
+        <command_interface name="position">          <!-- Add/Remove interfaces as needed -->
           <param name="min">-1</param>
           <param name="max">1</param>
@@ -92,47 +73,111 @@
         <state_interface name="acceleration"/>
       </joint>
-      <sensor name="tcp_fts_sensor">            <!-- Remove/change sensors as needed -->
-        <state_interface name="fx"/>
-        <state_interface name="fy"/>
-        <state_interface name="fz"/>
-        <state_interface name="tx"/>
-        <state_interface name="ty"/>
-        <state_interface name="tz"/>
-        <param name="frame_id">tool0</param>    <!-- Change sensors as needed -->
-        <param name="min_fx">-100</param>
-        <param name="max_fx">100</param>
-        <param name="min_fy">-100</param>
-        <param name="max_fy">100</param>
-        <param name="min_fz">-200</param>
-        <param name="max_fz">200</param>
-        <param name="min_tx">-10</param>
-        <param name="max_tx">10</param>
-        <param name="min_ty">-10</param>
-        <param name="max_ty">10</param>
-        <param name="min_tz">-15</param>
-        <param name="max_tz">15</param>
-      </sensor>
     </ros2_control>
-    <xacro:if value="$(arg sim_gazebo_classic)">
-      <!-- Gazebo plugins -->
-      <gazebo reference="world">
-      </gazebo>
-      <gazebo>
-        <plugin filename="libgazebo_ros2_control.so" name="gazebo_ros2_control">
-          <parameters>${simulation_controllers}</parameters>
-        </plugin>
-      </gazebo>
-    </xacro:if>
-    <xacro:if value="$(arg sim_gazebo)">
-      <!-- Gazebo plugins -->
-      <gazebo reference="world">
-      </gazebo>
-      <gazebo>
-        <plugin filename="libign_ros2_control-system.so" name="ign_ros2_control::IgnitionROS2ControlPlugin">
-          <parameters>${simulation_controllers}</parameters>
-          <controller_manager_node_name>${prefix}controller_manager</controller_manager_node_name>
-        </plugin>
-      </gazebo>
-    </xacro:if>
+    <!-- ========================================= -->
+    <!--  -->
+    <!-- ========================================= -->
+    <ros2_control name="ec_cool_robot" type="system">
+      <hardware>
+        <plugin>ethercat_driver/EthercatDriver</plugin>
+        <param name="master_id">0</param>
+        <param name="control_frequency">200</param>
+      </hardware>
+      <!-- joint1 -->
+      <joint name="${prefix}joint1">
+        <command_interface name="control_word"/>
+        <command_interface name="position"/>
+        <state_interface name="status_word"/>
+        <state_interface name="position"/>
+        <state_interface name="velocity"/>
+        <state_interface name="effort"/>
+        <ec_module name="RSM90E7_J1">
+          <plugin>ethercat_generic_plugins/EcCiA402Drive</plugin>
+          <param name="alias">0</param>
+          <param name="position">0</param>
+          <param name="mode_of_operation">8</param>
+          <param name="slave_config">(find cool_robot_description)/config/rs_m90e7.yaml</param>
+        </ec_module>
+      </joint>
+      <!-- joint2 -->
+      <joint name="${prefix}joint2">
+        <command_interface name="control_word"/>
+        <command_interface name="position"/>
+        <state_interface name="status_word"/>
+        <state_interface name="position"/>
+        <state_interface name="velocity"/>
+        <state_interface name="effort"/>
+        <ec_module name="RSM90E7_J1">
+          <plugin>ethercat_generic_plugins/EcCiA402Drive</plugin>
+          <param name="alias">0</param>
+          <param name="position">0</param>
+          <param name="mode_of_operation">8</param>
+          <param name="slave_config">(find cool_robot_description)/config/rs_m90e7.yaml</param>
+        </ec_module>
+      </joint>
+      <!-- joint3 -->
+      <joint name="${prefix}joint3">
+        <command_interface name="control_word"/>
+        <command_interface name="position"/>
+        <state_interface name="status_word"/>
+        <state_interface name="position"/>
+        <state_interface name="velocity"/>
+        <state_interface name="effort"/>
+        <ec_module name="RSM90E7_J1">
+          <plugin>ethercat_generic_plugins/EcCiA402Drive</plugin>
+          <param name="alias">0</param>
+          <param name="position">0</param>
+          <param name="mode_of_operation">8</param>
+          <param name="slave_config">(find cool_robot_description)/config/rs_m90e7.yaml</param>
+        </ec_module>
+      </joint>
+      <!-- joint4 -->
+      <joint name="${prefix}joint4">
+        <command_interface name="control_word"/>
+        <command_interface name="position"/>
+        <state_interface name="status_word"/>
+        <state_interface name="position"/>
+        <state_interface name="velocity"/>
+        <state_interface name="effort"/>
+        <ec_module name="RSM90E7_J1">
+          <plugin>ethercat_generic_plugins/EcCiA402Drive</plugin>
+          <param name="alias">0</param>
+          <param name="position">0</param>
+          <param name="mode_of_operation">8</param>
+          <param name="slave_config">(find cool_robot_description)/config/rs_m90e7.yaml</param>
+        </ec_module>
+      </joint>
+      <!-- joint5 -->
+      <joint name="${prefix}joint5">
+        <command_interface name="control_word"/>
+        <command_interface name="position"/>
+        <state_interface name="status_word"/>
+        <state_interface name="position"/>
+        <state_interface name="velocity"/>
+        <state_interface name="effort"/>
+        <ec_module name="RSM90E7_J1">
+          <plugin>ethercat_generic_plugins/EcCiA402Drive</plugin>
+          <param name="alias">0</param>
+          <param name="position">0</param>
+          <param name="mode_of_operation">8</param>
+          <param name="slave_config">(find cool_robot_description)/config/rs_m90e7.yaml</param>
+        </ec_module>
+      </joint>
+      <!-- joint6 -->
+      <joint name="${prefix}joint6">
+        <command_interface name="control_word"/>
+        <command_interface name="position"/>
+        <state_interface name="status_word"/>
+        <state_interface name="position"/>
+        <state_interface name="velocity"/>
+        <state_interface name="effort"/>
+        <ec_module name="RSM90E7_J1">
+          <plugin>ethercat_generic_plugins/EcCiA402Drive</plugin>
+          <param name="alias">0</param>
+          <param name="position">0</param>
+          <param name="mode_of_operation">8</param>
+          <param name="slave_config">(find cool_robot_description)/config/rs_m90e7.yaml</param>
+        </ec_module>
+      </joint>
+    </ros2_control>
   </xacro:macro>
 </robot>
