Commit message: control_manager不會當了 執行 ros2 launch cool_robot_bringup cool_robot.launch.py 之後 使用 ros2 control list_hardware_interfaces 可以列出訊息

File: cool_robot_description/urdf/cool_robot/cool_robot_macro.ros2_control.xacro (robot description, xacro)
@@ -4,74 +4,4 @@
                name
                prefix">
-    <ros2_control name="${name}" type="system">
-      <hardware>
-      </hardware>
-      <joint name="${prefix}joint1">
-        <command_interface name="position">          <!-- Add/Remove interfaces as needed -->
-          <param name="min">-1</param>
-          <param name="max">1</param>
-        </command_interface>
-        <state_interface name="position">
-          <param name="initial_value">0.0</param>
-        </state_interface>
-        <state_interface name="velocity"/>
-        <state_interface name="acceleration"/>
-      </joint>
-      <joint name="${prefix}joint2">
-        <command_interface name="position">          <!-- Add/Remove interfaces as needed -->
-          <param name="min">-1</param>
-          <param name="max">1</param>
-        </command_interface>
-        <state_interface name="position">
-          <param name="initial_value">0.0</param>
-        </state_interface>
-        <state_interface name="velocity"/>
-        <state_interface name="acceleration"/>
-      </joint>
-      <joint name="${prefix}joint3">
-        <command_interface name="position">          <!-- Add/Remove interfaces as needed -->
-          <param name="min">-1</param>
-          <param name="max">1</param>
-        </command_interface>
-        <state_interface name="position">
-          <param name="initial_value">0.0</param>
-        </state_interface>
-        <state_interface name="velocity"/>
-        <state_interface name="acceleration"/>
-      </joint>
-      <joint name="${prefix}joint4">
-        <command_interface name="position">          <!-- Add/Remove interfaces as needed -->
-          <param name="min">-1</param>
-          <param name="max">1</param>
-        </command_interface>
-        <state_interface name="position">
-          <param name="initial_value">0.0</param>
-        </state_interface>
-        <state_interface name="velocity"/>
-        <state_interface name="acceleration"/>
-      </joint>
-      <joint name="${prefix}joint5">
-        <command_interface name="position">          <!-- Add/Remove interfaces as needed -->
-          <param name="min">-1</param>
-          <param name="max">1</param>
-        </command_interface>
-        <state_interface name="position">
-          <param name="initial_value">0.0</param>
-        </state_interface>
-        <state_interface name="velocity"/>
-        <state_interface name="acceleration"/>
-      </joint>
-      <joint name="${prefix}joint6">
-        <command_interface name="position">          <!-- Add/Remove interfaces as needed -->
-          <param name="min">-1</param>
-          <param name="max">1</param>
-        </command_interface>
-        <state_interface name="position">
-          <param name="initial_value">0.0</param>
-        </state_interface>
-        <state_interface name="velocity"/>
-        <state_interface name="acceleration"/>
-      </joint>
-    </ros2_control>
     <!-- ========================================= -->
     <!--  -->
@@ -83,8 +13,11 @@
         <param name="control_frequency">200</param>
       </hardware>
+      <!-- ========================================= -->
       <!-- joint1 -->
+      <!-- ========================================= -->
       <joint name="${prefix}joint1">
         <command_interface name="control_word"/>
         <command_interface name="position"/>
+        <command_interface name="effort"/>
         <state_interface name="status_word"/>
         <state_interface name="position"/>
@@ -96,85 +29,100 @@
           <param name="position">0</param>
           <param name="mode_of_operation">8</param>
-          <param name="slave_config">(find cool_robot_description)/config/rs_m90e7.yaml</param>
+          <param name="slave_config">$(find cool_robot_description)/config/rs_m90e7.yaml</param>
         </ec_module>
       </joint>
+      <!-- ========================================= -->
       <!-- joint2 -->
+      <!-- ========================================= -->
       <joint name="${prefix}joint2">
         <command_interface name="control_word"/>
         <command_interface name="position"/>
+        <command_interface name="effort"/>
         <state_interface name="status_word"/>
         <state_interface name="position"/>
         <state_interface name="velocity"/>
         <state_interface name="effort"/>
-        <ec_module name="RSM90E7_J1">
+        <ec_module name="RSM90E7_J2">
           <plugin>ethercat_generic_plugins/EcCiA402Drive</plugin>
           <param name="alias">0</param>
-          <param name="position">0</param>
+          <param name="position">1</param>
           <param name="mode_of_operation">8</param>
-          <param name="slave_config">(find cool_robot_description)/config/rs_m90e7.yaml</param>
+          <param name="slave_config">$(find cool_robot_description)/config/rs_m90e7.yaml</param>
         </ec_module>
       </joint>
+      <!-- ========================================= -->
       <!-- joint3 -->
+      <!-- ========================================= -->
       <joint name="${prefix}joint3">
         <command_interface name="control_word"/>
         <command_interface name="position"/>
+        <command_interface name="effort"/>
         <state_interface name="status_word"/>
         <state_interface name="position"/>
         <state_interface name="velocity"/>
         <state_interface name="effort"/>
-        <ec_module name="RSM90E7_J1">
+        <ec_module name="RSM90E7_J3">
           <plugin>ethercat_generic_plugins/EcCiA402Drive</plugin>
           <param name="alias">0</param>
-          <param name="position">0</param>
+          <param name="position">2</param>
           <param name="mode_of_operation">8</param>
-          <param name="slave_config">(find cool_robot_description)/config/rs_m90e7.yaml</param>
+          <param name="slave_config">$(find cool_robot_description)/config/rs_m90e7.yaml</param>
         </ec_module>
       </joint>
+      <!-- ========================================= -->
       <!-- joint4 -->
+      <!-- ========================================= -->
       <joint name="${prefix}joint4">
         <command_interface name="control_word"/>
         <command_interface name="position"/>
+        <command_interface name="effort"/>
         <state_interface name="status_word"/>
         <state_interface name="position"/>
         <state_interface name="velocity"/>
         <state_interface name="effort"/>
-        <ec_module name="RSM90E7_J1">
+        <ec_module name="RSM90E7_J4">
           <plugin>ethercat_generic_plugins/EcCiA402Drive</plugin>
           <param name="alias">0</param>
-          <param name="position">0</param>
+          <param name="position">3</param>
           <param name="mode_of_operation">8</param>
-          <param name="slave_config">(find cool_robot_description)/config/rs_m90e7.yaml</param>
+          <param name="slave_config">$(find cool_robot_description)/config/rs_m90e7.yaml</param>
         </ec_module>
       </joint>
+      <!-- ========================================= -->
       <!-- joint5 -->
+      <!-- ========================================= -->
       <joint name="${prefix}joint5">
         <command_interface name="control_word"/>
         <command_interface name="position"/>
+        <command_interface name="effort"/>
         <state_interface name="status_word"/>
         <state_interface name="position"/>
         <state_interface name="velocity"/>
         <state_interface name="effort"/>
-        <ec_module name="RSM90E7_J1">
+        <ec_module name="RSM90E7_J5">
           <plugin>ethercat_generic_plugins/EcCiA402Drive</plugin>
           <param name="alias">0</param>
-          <param name="position">0</param>
+          <param name="position">4</param>
           <param name="mode_of_operation">8</param>
-          <param name="slave_config">(find cool_robot_description)/config/rs_m90e7.yaml</param>
+          <param name="slave_config">$(find cool_robot_description)/config/rs_m90e7.yaml</param>
         </ec_module>
       </joint>
+      <!-- ========================================= -->
       <!-- joint6 -->
+      <!-- ========================================= -->
       <joint name="${prefix}joint6">
         <command_interface name="control_word"/>
         <command_interface name="position"/>
+        <command_interface name="effort"/>
         <state_interface name="status_word"/>
         <state_interface name="position"/>
         <state_interface name="velocity"/>
         <state_interface name="effort"/>
-        <ec_module name="RSM90E7_J1">
+        <ec_module name="RSM90E7_J6">
           <plugin>ethercat_generic_plugins/EcCiA402Drive</plugin>
           <param name="alias">0</param>
-          <param name="position">0</param>
+          <param name="position">5</param>
           <param name="mode_of_operation">8</param>
-          <param name="slave_config">(find cool_robot_description)/config/rs_m90e7.yaml</param>
+          <param name="slave_config">$(find cool_robot_description)/config/rs_m90e7.yaml</param>
         </ec_module>
       </joint>
